File: output_folder/pcbs/base.kicad_pcb (KiCad board)
At the start: 2 copper layers, 257 x 154.6 mm, 125 parts

Commit message: basic outline ready
Parts:
- removed LED39, LED40, LED41, LED42, LED43, LED44, LED45, LED46: , ceoloide:YS-SK6812MINI-E (per-key, reversible)
- removed S39, S40, S41, S42, S43, S44, S45, S46: , PG1350
- added D31: , ComboDiode, F.Cu at (209.2, 138.0)
- added D32: , ComboDiode, F.Cu at (214.3, 181.9)
- added D33: , ComboDiode, F.Cu at (204.3, 165.8)
- added D34: , ComboDiode, F.Cu at (194.2, 149.7)
- added D35: , ComboDiode, F.Cu at (227.8, 195.9)
- added D36: , ComboDiode, F.Cu at (213.9, 212.4)
- added D37: , ComboDiode, F.Cu at (205.6, 232.2)
- added D38: , ComboDiode, F.Cu at (199.1, 200.1)
- moved D18 156.2 mm to (167.7, 232.2), turned to 22 degrees
- moved D16 148.2 mm to (145.5, 195.9), turned to 58 degrees
- moved S20 147.6 mm to (298.6, 160.2), turned to -168 degrees
- moved LED20 144.1 mm to (297.6, 155.6), turned to 12 degrees
- moved D17 143.7 mm to (159.4, 212.4), turned to 40 degrees
- moved S22 140.0 mm to (290.7, 123.0), turned to -168 degrees
- moved LED22 136.9 mm to (289.7, 118.4), turned to 12 degrees
- moved S21 134.5 mm to (294.7, 141.6), turned to -168 degrees
- moved LED21 131.7 mm to (293.7, 137.0), turned to 12 degrees
- moved D19 102.6 mm to (174.2, 200.1), turned to 40 degrees
- moved S23 95.1 mm to (273.7, 149.5), turned to -158 degrees
- moved LED23 90.5 mm to (272.0, 145.2), turned to 22 degrees
- moved D28 66.4 mm to (225.0, 116.4), turned to 117 degrees
- moved LED32 66.1 mm to (218.9, 172.3), turned to 32 degrees
- moved S32 65.8 mm to (221.4, 176.3), turned to -148 degrees
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Connections:
- D16 pad 1: R1 -> P9
- D16 pad 2: mirror_pinky_bottom -> near_thumb
- D17 pad 1: R2 -> P9
- D17 pad 2: mirror_pinky_home -> home_thumb
- D18 pad 1: R3 -> P9
- D18 pad 2: mirror_pinky_top -> far_thumb
- D19 pad 1: R1 -> P9
- D19 pad 2: mirror_ring_bottom -> home_thumb
- D20 pad 1: R2 -> R1
- D20 pad 2: mirror_ring_home -> mirror_pinky_bottom
- D21 pad 1: R3 -> R2
- D21 pad 2: mirror_ring_top -> mirror_pinky_home
- D22 pad 1: R1 -> R3
- D22 pad 2: mirror_middle_bottom -> mirror_pinky_top
- D23 pad 1: R2 -> R1
- D23 pad 2: mirror_middle_home -> mirror_ring_bottom
- D24 pad 1: R3 -> R2
- D24 pad 2: mirror_middle_top -> mirror_ring_home
- D25 pad 1: R1 -> R3
- D25 pad 2: mirror_index_bottom -> mirror_ring_top
- D26 pad 1: R2 -> R1
- D26 pad 2: mirror_index_home -> mirror_middle_bottom
- D27 pad 1: R3 -> R2
- D27 pad 2: mirror_index_top -> mirror_middle_home
- D28 pad 1: R1 -> R3
- D28 pad 2: mirror_inner_bottom -> mirror_middle_top
- D29 pad 1: R2 -> R1
- D29 pad 2: mirror_inner_home -> mirror_index_bottom
- D30 pad 1: R3 -> R2
- D30 pad 2: mirror_inner_top -> mirror_index_home
- LED16 pad 2: (no net) -> LED_20
- LED16 pad 4: (no net) -> LED_19
- LED18 pad 2: (no net) -> LED_23
- LED18 pad 4: (no net) -> LED_22
- LED19 pad 2: LED_20 -> ULED_6
- LED19 pad 4: LED_19 -> LED_24
- LED20 pad 2: (no net) -> LED_4
- LED20 pad 4: (no net) -> LED_3
- LED21 pad 2: LED_23 -> LED_3
- LED21 pad 4: LED_22 -> LED_2
- LED22 pad 2: (no net) -> LED_2
- LED22 pad 4: (no net) -> LED_1
- LED23 pad 2: ULED_6 -> LED_5
- LED23 pad 4: LED_24 -> LED_4
- LED24 pad 2: LED_4 -> LED_6
- LED24 pad 4: LED_3 -> LED_5
- LED25 pad 2: LED_3 -> LED_7
- LED25 pad 4: LED_2 -> LED_6
- LED26 pad 2: LED_2 -> LED_10
- LED26 pad 4: LED_1 -> LED_9
- LED27 pad 2: LED_5 -> LED_9
- LED27 pad 4: LED_4 -> LED_8
- LED28 pad 2: LED_6 -> LED_8
- LED28 pad 4: LED_5 -> LED_7
- LED29 pad 2: LED_7 -> LED_13
- LED29 pad 4: LED_6 -> LED_12
- LED30 pad 2: LED_10 -> LED_11
- LED30 pad 4: LED_9 -> LED_12
- LED31 pad 2: LED_9 -> LED_10
- LED31 pad 4: LED_8 -> LED_11
- LED32 pad 2: LED_8 -> LED_14
- LED32 pad 4: LED_7 -> LED_13
- LED33 pad 2: LED_13 -> LED_15
- LED33 pad 4: LED_12 -> LED_14
- LED34 pad 2: LED_11 -> LED_17
- LED34 pad 4: LED_12 -> LED_16
- LED35 pad 2: LED_10 -> LED_20
- LED35 pad 4: LED_11 -> LED_19
- LED36 pad 2: LED_14 -> LED_20
- LED36 pad 4: LED_13 -> LED_19
- LED37 pad 2: LED_15 -> LED_23
- LED37 pad 4: LED_14 -> LED_22
- LED38 pad 2: LED_17 -> ULED_6
- LED38 pad 4: LED_16 -> LED_24
- S17 pad 1: SDA -> SLC
- S17 pad 2: near_bottom -> home_thumb
- S18 pad 1: SLC -> CS
- S18 pad 2: home_thumb -> far_thumb
- S19 pad 1: SLC -> R0
- S19 pad 2: home_bottom -> home_thumb
- S20 pad 1: CS -> P10
- S20 pad 2: far_thumb -> mirror_pinky_bottom
- S21 pad 1: CS -> P10
- S21 pad 2: far_bottom -> mirror_pinky_home
- S22 pad 1: R0 -> P10
- S22 pad 2: home_thumb -> mirror_pinky_top
- S23 pad 1: R0 -> C0
- S23 pad 2: home_home -> mirror_ring_bottom
- S24 pad 1: P10 -> C0
- S24 pad 2: mirror_pinky_bottom -> mirror_ring_home
- S25 pad 1: P10 -> C0
- S25 pad 2: mirror_pinky_home -> mirror_ring_top
- S26 pad 1: P10 -> C1
- S26 pad 2: mirror_pinky_top -> mirror_middle_bottom
- S27 pad 1: C0 -> C1
- S27 pad 2: mirror_ring_bottom -> mirror_middle_home
- S28 pad 1: C0 -> C1
- S28 pad 2: mirror_ring_home -> mirror_middle_top
- S29 pad 1: C0 -> C2
- S29 pad 2: mirror_ring_top -> mirror_index_bottom
- S30 pad 1: C1 -> C2
- S30 pad 2: mirror_middle_bottom -> mirror_index_home
- S31 pad 1: C1 -> C2
- S31 pad 2: mirror_middle_home -> mirror_index_top
- S32 pad 1: C1 -> C3
- S32 pad 2: mirror_middle_top -> mirror_inner_bottom
- S33 pad 1: C2 -> C3
- S33 pad 2: mirror_index_bottom -> mirror_inner_home
- S34 pad 1: C2 -> C3
- S34 pad 2: mirror_index_home -> mirror_inner_top
- S35 pad 1: C2 -> C4
- S35 pad 2: mirror_index_top -> mirror_near_thumb
- S36 pad 1: C3 -> C5
- S36 pad 2: mirror_inner_bottom -> mirror_home_thumb
- S37 pad 1: C3 -> P16
- S37 pad 2: mirror_inner_home -> mirror_far_thumb
- S38 pad 1: C3 -> P10
- S38 pad 2: mirror_inner_top -> mirror_home_thumb
Routing:
- net (no net): track 108.2 -> 0.00 mm, vias 16 -> 0
- net home_bottom: track 50.9 -> 0.00 mm
- net P10: track 0.00 -> 50.9 mm
- net home_thumb: track 50.9 -> 0.00 mm
- net far_thumb: track 0.00 -> 50.9 mm
- net GND: track 172.7 -> 142.7 mm, vias 46 -> 38
- net VCC: track 172.7 -> 142.7 mm, vias 46 -> 38
