File: output_folder/pcbs/main.kicad_pcb (KiCad board)
At the start: 2 copper layers, 257 x 154.6 mm, 117 parts

Commit message: messing around
Parts:
- added D39: , ComboDiode, F.Cu at (186.7, 186.3)
- added ROT1: , rotary_encoder, F.Cu at (186.7, 171.3)
Connections:
- LED10 pad 2: LED_13 -> LED_11
- LED10 pad 4: LED_12 -> LED_10
- LED11 pad 2: LED_11 -> LED_12
- LED11 pad 4: LED_12 -> LED_11
- LED12 pad 2: LED_10 -> LED_13
- LED12 pad 4: LED_11 -> LED_12
- LED13 pad 2: LED_14 -> LED_16
- LED13 pad 4: LED_13 -> LED_15
- LED15 pad 2: LED_17 -> LED_14
- LED15 pad 4: LED_16 -> LED_13
- LED16 pad 2: LED_20 -> LED_17
- LED16 pad 4: LED_19 -> LED_16
- LED17 pad 2: LED_20 -> LED_18
- LED17 pad 4: LED_19 -> LED_17
- LED18 pad 2: LED_23 -> LED_20
- LED18 pad 4: LED_22 -> LED_19
- LED19 pad 2: ULED_6 -> LED_19
- LED19 pad 4: LED_24 -> LED_18
- LED20 pad 2: LED_4 -> LED_37
- LED20 pad 4: LED_3 -> LED_36
- LED21 pad 2: LED_3 -> LED_38
- LED21 pad 4: LED_2 -> LED_37
- LED22 pad 2: LED_2 -> (no net)
- LED22 pad 4: LED_1 -> LED_38
- LED23 pad 2: LED_5 -> LED_36
- LED23 pad 4: LED_4 -> LED_35
- LED24 pad 2: LED_6 -> LED_35
- LED24 pad 4: LED_5 -> LED_34
- LED25 pad 2: LED_7 -> LED_34
- LED25 pad 4: LED_6 -> LED_33
- LED26 pad 2: LED_10 -> LED_31
- LED26 pad 4: LED_9 -> LED_30
- LED27 pad 2: LED_9 -> LED_32
- LED27 pad 4: LED_8 -> LED_31
- LED28 pad 2: LED_8 -> LED_33
- LED28 pad 4: LED_7 -> LED_32
- LED29 pad 2: LED_13 -> LED_30
- LED29 pad 4: LED_12 -> LED_29
- LED3 pad 4: LED_1 -> LED
- LED30 pad 2: LED_11 -> LED_29
- LED30 pad 4: LED_12 -> LED_28
- LED31 pad 2: LED_10 -> LED_28
- LED31 pad 4: LED_11 -> LED_27
- LED32 pad 2: LED_14 -> LED_25
- LED32 pad 4: LED_13 -> LED_24
- LED33 pad 2: LED_15 -> LED_26
- LED33 pad 4: LED_14 -> LED_25
- LED34 pad 2: LED_17 -> LED_27
- LED34 pad 4: LED_16 -> LED_26
- LED35 pad 2: LED_20 -> LED_24
- LED35 pad 4: LED_19 -> LED_23
- LED36 pad 2: LED_20 -> LED_23
- LED36 pad 4: LED_19 -> LED_22
- LED37 pad 2: LED_23 -> LED_21
- LED37 pad 4: LED_22 -> LED_20
- LED38 pad 2: ULED_6 -> LED_22
- LED38 pad 4: LED_24 -> LED_21
Routing:
- net DAT: track 121.9 -> 0.00 mm
- net CS: track 121.8 -> 0.00 mm
- net P10: track 50.9 -> 0.00 mm
- net far_thumb: track 50.9 -> 0.00 mm
- net LED_28: track 0.00 -> 13.5 mm, vias 0 -> 2
- net LED_4: track 27.1 -> 13.5 mm, vias 4 -> 2
- net LED_36: track 0.00 -> 13.5 mm, vias 0 -> 2
- net LED_33: track 0.00 -> 13.5 mm, vias 0 -> 2
- net LED_7: track 27.1 -> 13.5 mm, vias 4 -> 2
- net LED_10: track 27.1 -> 13.5 mm, vias 4 -> 2
- net LED_21: track 0.00 -> 13.5 mm, vias 0 -> 2
- net LED_5: track 27.1 -> 13.5 mm, vias 4 -> 2
- net LED_37: track 0.00 -> 13.5 mm, vias 0 -> 2
- net LED_11: track 27.1 -> 13.5 mm, vias 4 -> 2
- net LED_34: track 0.00 -> 13.5 mm, vias 0 -> 2
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Other:
- board size 257 x 154.6 mm -> 246.9 x 153.3 mm
