File: archaeoptereeks/output_folder2/pcbs/_autosave-main_r1.kicad_pcb (KiCad board)
At the start: 2 copper layers, 246.9 x 153.3 mm, 111 parts

Commit message: adding mounting holes and top plate
Parts:
- moved D5 44.7 mm to (76.2, 162.0)
- moved S32 44.7 mm to (172.8, 186.0)
- moved LED3 44.7 mm to (45.1, 144.2)
- moved D34 44.7 mm to (189.3, 221.7)
- moved LED7 44.7 mm to (87.1, 166.9)
- moved LED26 44.7 mm to (200.5, 149.9)
- moved D2 44.7 mm to (48.7, 170.2)
- moved D23 44.7 mm to (220.1, 162.0)
- moved D10 44.7 mm to (105.4, 195.9)
- moved D29 44.7 mm to (180.8, 179.8)
- moved LED30 44.7 mm to (175.3, 154.1)
- moved LED32 44.7 mm to (170.3, 182.0)
- moved LED33 44.7 mm to (160.3, 165.9)
- moved LED29 44.7 mm to (185.4, 170.2)
- moved S31 44.7 mm to (182.9, 202.1)
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Routing:
- net C0: track 479.3 -> 563.7 mm
- net VCC: track 1408.4 -> 1459.9 mm, vias 36 -> 37
- net mirror_far_thumb: track 2.16 -> 13.9 mm
- net mirror_home_thumb: track 2.16 -> 13.9 mm
- net P9: track 349.1 -> 354.8 mm
- net C3: track 180.4 -> 185.3 mm
- net R2: track 296.0 -> 299.7 mm
- net R3: track 162.9 -> 165.4 mm
- net GND: track 1496.4 -> 1499.0 mm
- net C4: track 268.0 -> 270.4 mm
- net R1: track 275.7 -> 278.1 mm
- net C1: track 486.0 -> 488.4 mm
- net RST: track 54.9 -> 57.1 mm
- net C2: track 288.5 -> 290.7 mm
- net R0: track 331.9 -> 333.4 mm
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- added copper zone on B.Cu, net GND
- added copper zone on F.Cu, net GND
