File: archaeoptereeks/output_folder2/pcbs/main_routed.kicad_pcb (KiCad board)
At the start: 2 copper layers, 246.9 x 153.3 mm, 111 parts

Commit message: adding mounting holes and top plate
Parts:
- moved D19 10.5 mm to (274.1, 161.5)
- moved S28 10.5 mm to (220.6, 163.0)
- moved D15 10.5 mm to (163.2, 148.1)
- moved D29 10.5 mm to (203.4, 152.5)
- moved LED27 10.5 mm to (214.5, 105.7)
- moved S12 10.5 mm to (141.1, 130.7)
- moved D6 10.5 mm to (105.9, 117.0)
- moved B1 10.5 mm to (185.1, 98.1)
- moved B2 10.5 mm to (185.1, 98.1)
- moved LED3 10.5 mm to (67.7, 116.8)
- moved D34 10.5 mm to (211.9, 194.3)
- moved LED11 10.5 mm to (133.5, 142.9)
- moved LED22 10.5 mm to (256.1, 143.6)
- moved LED25 10.5 mm to (231.8, 139.5)
- moved LED30 10.5 mm to (197.9, 126.8)
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Routing:
- net GND: track 1496.4 -> 1505.2 mm
- net RST: track 54.9 -> 63.6 mm
