File: archaeoptereeks/output_folder2/pcbs/archaeoptereeks.kicad_pcb (KiCad board)
At the start: 2 copper layers, 246.9 x 153.3 mm, 111 parts

Commit message: playing with ergogen and working on silk drawings
Parts:
- added H1: , mounting_hole, F.Cu at (98.8, 104.5)
- added H2: , mounting_hole, F.Cu at (274.9, 104.5)
- added H3: , mounting_hole, F.Cu at (160.6, 110.0)
- added H4: , mounting_hole, F.Cu at (213.1, 110.0)
- added H5: , mounting_hole, F.Cu at (89.5, 162.9)
- added H6: , mounting_hole, F.Cu at (284.2, 162.9)
- added H7: , mounting_hole, F.Cu at (177.6, 229.2)
- added H8: , mounting_hole, F.Cu at (196.1, 229.2)
- added REF**: Testout_edge_4, KiCadLibs:Testout_edge_4, F.Cu at (176.2, 163.6)
- moved LED27 49.8 mm to (230.6, 101.7)
- moved S24 49.8 mm to (259.7, 108.7)
- moved LED31 49.8 mm to (219.1, 166.8)
- moved LED29 49.8 mm to (224.1, 138.9)
- moved S14 49.8 mm to (162.2, 154.6)
- moved S19 49.8 mm to (298.8, 154.6)
- moved S17 49.8 mm to (154.6, 199.3)
- moved LED25 49.8 mm to (247.8, 135.5)
- moved S32 49.8 mm to (211.5, 154.6)
- moved LED34 49.8 mm to (232.6, 180.8)
- moved D27 49.8 mm to (225.2, 110.8)
- moved D7 49.8 mm to (131.3, 144.7)
- moved D35 49.8 mm to (214.1, 206.8)
- moved LED3 49.8 mm to (83.8, 112.9)
- moved LED36 49.8 mm to (203.9, 216.2)
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Routing:
- net GND: track 1499.0 -> 1686.2 mm, vias 39 -> 45
- net VCC: track 1459.9 -> 1584.2 mm, vias 37 -> 42
- net SDA: track 14.1 -> 108.3 mm, vias 0 -> 2
- net SCL: track 14.1 -> 108.0 mm, vias 0 -> 2
- net RST: track 57.1 -> 0.00 mm, vias 1 -> 0
- net C4: track 270.4 -> 254.0 mm
- net P10: track 237.7 -> 253.6 mm
- net C0: track 563.7 -> 547.9 mm
- net P16: track 294.4 -> 310.2 mm
- net C5: track 256.9 -> 271.6 mm
- net MCU1_5: track 8.50 -> 22.6 mm
- net MCU1_1: track 8.48 -> 22.6 mm
- net RAW: track 14.1 -> 0.00 mm
- net MCU1_8: track 8.45 -> 22.6 mm
- net MCU1_6: track 8.48 -> 22.6 mm
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- added copper zone on B.Cu, net VCC
- removed copper zone on B.Cu, net GND
Other:
- board text added: "JLCJLCJLCJLC"
