File: archaeoptereeks/output_folder2/pcbs/main_r2.kicad_pcb (KiCad board)
At the start: 2 copper layers, 246.9 x 153.3 mm, 119 parts

Commit message: playing with ergogen and working on silk drawings
Parts:
- moved H5 49.3 mm to (48.0, 177.6)
- moved D7 49.3 mm to (89.8, 159.5)
- moved D5 49.3 mm to (73.4, 145.4)
- moved D9 49.3 mm to (107.1, 125.6)
- moved H3 49.3 mm to (119.1, 124.8)
- moved LED14 49.3 mm to (123.2, 165.4)
- moved LED30 49.3 mm to (172.6, 137.6)
- moved S19 49.3 mm to (257.3, 169.4)
- moved D10 49.3 mm to (102.7, 179.4)
- moved D26 49.3 mm to (192.3, 142.6)
- moved D32 49.3 mm to (163.0, 175.1)
- moved D34 49.3 mm to (186.5, 205.2)
- moved D18 49.3 mm to (126.4, 241.4)
- moved LED13 49.3 mm to (113.1, 181.6)
- moved S18 49.3 mm to (124.0, 232.7)
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Routing:
- net VCC: track 1459.3 -> 1569.3 mm, vias 37 -> 39
- net GND: track 1578.8 -> 1673.3 mm, vias 43 -> 44
- net SDA: track 14.1 -> 91.4 mm, vias 0 -> 1
- net SCL: track 14.1 -> 87.0 mm, vias 0 -> 1
- net C0: track 563.7 -> 547.9 mm
- net C4: track 268.5 -> 254.4 mm
- net MCU1_5: track 8.50 -> 22.6 mm
- net MCU1_1: track 8.48 -> 22.6 mm
- net RAW: track 14.1 -> 0.00 mm
- net MCU1_8: track 8.45 -> 22.6 mm
- net MCU1_6: track 8.48 -> 22.6 mm
- net MCU1_7: track 8.50 -> 22.6 mm
- net MCU1_9: track 8.48 -> 22.6 mm
- net C3: track 185.3 -> 171.6 mm
- net C2: track 293.4 -> 287.4 mm
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Other:
- outline, holes or cut-outs redrawn
